File: KiCad/2mppt setup/MPPT.kicad_sch (KiCad schematic)
At the start: 2 parts

Commit message: Fix wiring check issue
Changed lines of the file:
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@@
-	(wire
-		(pts
-			(xy 139.7 85.09) (xy 134.62 85.09)
-		)
-		(stroke
-			(width 0)
-			(type default)
-		)
-	)
 	(wire
 		(pts
@@
 	(wire
 		(pts
-			(xy 127 85.09) (xy 124.46 85.09)
+			(xy 125.73 85.09) (xy 124.46 85.09)
 		)
 		(stroke
@@
 	(wire
 		(pts
+			(xy 124.46 87.63) (xy 139.7 87.63)
+		)
+		(stroke
+			(width 0)
+			(type default)
+		)
+	)
+	(wire
+		(pts
 			(xy 139.7 93.98) (xy 124.46 93.98)
 		)
@@
 	(wire
 		(pts
+			(xy 133.35 85.09) (xy 139.7 85.09)
+		)
+		(stroke
+			(width 0)
+			(type default)
+		)
+	)
+	(wire
+		(pts
 			(xy 139.7 109.22) (xy 124.46 109.22)
 		)
@@
 		(pts
 			(xy 139.7 102.87) (xy 124.46 102.87)
-		)
-		(stroke
-			(width 0)
-			(type default)
-		)
-	)
-	(wire
-		(pts
-			(xy 139.7 87.63) (xy 124.46 87.63)
 		)
 		(stroke
@@
 	(symbol
 		(lib_id "Device:Fuse")
-		(at 130.81 85.09 90)
+		(at 129.54 85.09 90)
 		(unit 1)
 		(exclude_from_sim no)
@@
 		(dnp no)
 		(property "Reference" "F4"
-			(at 129.5399 82.55 0)
+			(at 128.2699 82.55 0)
 			(effects
 				(font
@@
 		)
 		(property "Value" "F1"
-			(at 132.842 82.804 90)
+			(at 131.572 82.804 90)
 			(effects
 				(font
@@
 		)
 		(property "Footprint" ""
-			(at 130.81 86.868 90)
+			(at 129.54 86.868 90)
 			(effects
 				(font
@@
 		)
 		(property "Datasheet" "~"
-			(at 130.81 85.09 0)
+			(at 129.54 85.09 0)
 			(effects
 				(font
@@
 		)
 		(property "Description" "Fuse"
-			(at 130.81 85.09 0)
+			(at 129.54 85.09 0)
 			(effects
 				(font
@@
 		)
 		(property "Rating" "150% 100A = 150A"
-			(at 119.38 80.518 90)
+			(at 109.22 80.518 90)
 			(show_name yes)
 			(effects
