File: KiCad/2mppt setup/MPPT_MCU_TX.kicad_sch (KiCad schematic)
At the start: 8 parts, among them U1 ADS1115IDGS

Commit message: Fix wiring check issue
Changed lines of the file:
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@@
+	(wire
+		(pts
+			(xy 142.24 71.12) (xy 142.24 97.79)
+		)
+		(stroke
+			(width 0)
+			(type default)
+		)
+	)
 	(wire
 		(pts
@@
 		(pts
 			(xy 91.44 101.6) (xy 93.98 101.6)
-		)
-		(stroke
-			(width 0)
-			(type default)
-		)
-	)
-	(wire
-		(pts
-			(xy 142.24 97.79) (xy 142.24 71.12)
 		)
 		(stroke
@@
 	)
 	(symbol
-		(lib_name "ESP8266_custom_1")
 		(lib_id "Proa:ESP8266_custom")
 		(at 168.91 114.3 0)

Commit message: KiCad_Skip & Schemdraw test
Parts:
- removed DC-DC_Buck_Converter1: ~, symbol Proa:DC-DC_Buck_Converter
- added R6: 5.1k, symbol Device:R
- added R7: 10k, symbol Device:R
- added U2: BUCK_24V_5V_5A, symbol Proa:BUCK_24V_5V_5A
- R2, R5: value 1.1k -> 5.1k
- R3, R4: value 2.2k -> 10k
Connections:
- net 24V+: now also U2.2 (Vin-)
- net 24V-: now also U2.1 (Vin+)
- net AIN0: now also R6.2; no longer U1.4 (AIN0)
- net GND1: now also R7.2
- net at A1.20 (GND_(In)), A2.20 (GND_(In)): now also U2.4 (Vout-)
- net at A1.21 (VIN), A2.21 (VIN), U1.8 (VDD): now also U2.3 (Vout+)
- new net: R6.1, R7.1, U1.4 (AIN0)
