File: KiCad/test/test.kicad_sch (KiCad schematic)
At the start: 3 parts, among them U1 BUCK_24V_5V_5A

Commit message: setup kicad5 for skidl
Parts:
- removed R1: 1k, symbol Device:R
- removed U1: BUCK_24V_5V_5A, symbol Proa:BUCK_24V_5V_5A
- removed V1: 30, symbol Simulation_SPICE:VDC
