File: KiCad/Sensor Reader V3/mcu.kicad_sch (KiCad schematic)
At the start: 14 parts, among them J1 Conn_01x04_Socket, J3 Conn_01x02_Socket, J4 Conn_01x02_Socket, U3 ADS1115IDGS, U5 TCA9800

Commit message: Update sch
Parts:
- added C7: 0.1uF, symbol Device:C_Small
- C2: value 220uF -> 100uF
Connections:
- net 5V: now also C7.2
- net GND: now also C7.1
Other:
- moved on the sheet: J1, J3, R4, R5
