File: KiCad/Sensor Reader V3/Sensor Reader V3.kicad_sch (KiCad schematic)
At the start: 26 parts, among them J2 Conn_01x02_Pin, J5 Conn_01x04_Pin, J6 Conn_01x02_Pin, U1 BUCK_48V_24V_10A, U2 BUCK_24V_5V_5A

Commit message: Update sch
Parts:
- removed D1, D2: D_Small, symbol Device:D_Small
- added BT1: Battery, symbol Device:Battery
- added Fuse_4, Fuse_5: 100A, symbol Device:Fuse
- added SW1, SW2: SW_DIP_x02, symbol Switch:SW_DIP_x02
- Fuse_2, Fuse_3: value 100A -> 60A
Connections:
- net MPPT-_2 is gone; now on net MPPT-_1: SmartSolar_MPPT_150_1.3 (BATTERY-), SmartSolar_MPPT_150_1.9 (BODY_GND)
- net 48V+: now also SW1.3; no longer Li_ion(LiNMC)_Battery2.5 (Load+)
- net GND: now also SW2.4; no longer Li_ion(LiNMC)_Battery1.4 (Load-)
- net MPPT-_1: now also SW2.3
- net at Li_ion(LiNMC)_Battery1.3 (Charge-): now also SW2.2
- net at Fuse_1.2: now also SW1.4; no longer Li_ion(LiNMC)_Battery2.6 (Charge+)
- new net: Li_ion(LiNMC)_Battery1.4 (Load-), SW2.1
- new net: Fuse_4.1, SW1.2
- new net: Fuse_4.2, Li_ion(LiNMC)_Battery2.5 (Load+)
- new net: Li_ion(LiNMC)_Battery2.6 (Charge+), SW1.1
- new net: BT1.1 (+), Fuse_5.2
- no-connect marks 2 -> 6
Other:
- note added: "Spare Battery (LiFePo4)"
- moved on the sheet: Fuse_1, Fuse_2, Fuse_3, HE_Sensor_1, HE_Sensor_2, J2, J5, J6, Li_ion(LiNMC)_Battery1, Li_ion(LiNMC)_Battery2, R1

Commit message: Update kicad electrical schematics drawing
Connections:
- net MPPT-_1 is gone; now on net GND: SW2.3, SmartSolar_MPPT_150_1.3 (BATTERY-), SmartSolar_MPPT_150_1.9 (BODY_GND), SmartSolar_MPPT_150_2.3 (BATTERY-), SmartSolar_MPPT_150_2.9 (BODY_GND)
- net PV-_1 is gone; now on net GND: SmartSolar_MPPT_150_2.1 (PV+), TSM-NEG9R.28_6.2 (-), TSM-NEG9R.28_8.2 (-)
- net PV-_2 is gone; now on net GND: SmartSolar_MPPT_150_1.1 (PV+), TSM-NEG9R.28_1.2 (-), TSM-NEG9R.28_4.2 (-)
- net MPPT+_1 renamed mppt_output_1
- net MPPT+_2 renamed mppt_output_2
- net PV+_1 renamed solar_array_output_1
- net PV+_2 renamed solar_array_output_2
Other:
- moved on the sheet: Fuse_3
Changed lines of the file:
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@@
 	(wire
 		(pts
-			(xy 129.54 107.95) (xy 134.62 107.95)
+			(xy 128.27 107.95) (xy 133.35 107.95)
 		)
 		(stroke
@@
 	(wire
 		(pts
-			(xy 133.35 124.46) (xy 133.35 123.19)
+			(xy 132.08 124.46) (xy 132.08 123.19)
 		)
 		(stroke
@@
 	(wire
 		(pts
-			(xy 110.49 124.46) (xy 133.35 124.46)
+			(xy 110.49 124.46) (xy 132.08 124.46)
 		)
 		(stroke
@@
 	(wire
 		(pts
-			(xy 133.35 110.49) (xy 134.62 110.49)
+			(xy 132.08 110.49) (xy 133.35 110.49)
 		)
 		(stroke
@@
 	(wire
 		(pts
-			(xy 105.41 127) (xy 129.54 127)
-		)
-		(stroke
-			(width 0)
-			(type default)
-		)
-	)
-	(wire
-		(pts
-			(xy 133.35 110.49) (xy 133.35 115.57)
+			(xy 105.41 127) (xy 128.27 127)
+		)
+		(stroke
+			(width 0)
+			(type default)
+		)
+	)
+	(wire
+		(pts
+			(xy 132.08 110.49) (xy 132.08 115.57)
 		)
 		(stroke
@@
 	(wire
 		(pts
-			(xy 129.54 107.95) (xy 129.54 127)
-		)
-		(stroke
-			(width 0)
-			(type default)
-		)
-	)
-	(label "PV+_2"
+			(xy 128.27 107.95) (xy 128.27 127)
+		)
+		(stroke
+			(width 0)
+			(type default)
+		)
+	)
+	(label "solar_array_output_2"
 		(at 252.73 36.83 0)
 		(effects
@@
 		)
 	)
-	(label "MPPT-_1"
+	(label "GND"
 		(at 111.76 107.95 0)
 		(effects
@@
 		)
 	)
-	(label "MPPT+_2"
-		(at 134.62 110.49 0)
+	(label "mppt_output_2"
+		(at 133.35 110.49 0)
 		(effects
 			(font
@@
 		)
 	)
-	(label "MPPT+_1"
+	(label "mppt_output_1"
 		(at 111.76 110.49 0)
 		(effects
@@
 		)
 	)
-	(label "PV-_1"
+	(label "GND"
 		(at 110.49 31.75 0)
 		(effects
@@
 		)
 	)
-	(label "MPPT+_1"
+	(label "mppt_output_1"
 		(at 200.66 30.48 0)
 		(effects
@@
 		)
 	)
-	(label "PV+_2"
+	(label "solar_array_output_2"
 		(at 110.49 52.07 0)
 		(effects
@@
 		)
 	)
-	(label "PV+_1"
+	(label "solar_array_output_1"
 		(at 110.49 29.21 0)
 		(effects
@@
 		)
 	)
-	(label "PV-_2"
+	(label "GND"
 		(at 252.73 39.37 0)
 		(effects
@@
 		)
 	)
-	(label "MPPT+_2"
+	(label "mppt_output_2"
 		(at 252.73 30.48 0)
 		(effects
@@
 		)
 	)
-	(label "MPPT-_1"
+	(label "GND"
 		(at 200.66 33.02 0)
 		(effects
@@
 		)
 	)
-	(label "PV-_2"
+	(label "GND"
 		(at 110.49 54.61 0)
 		(effects
@@
 		)
 	)
-	(label "MPPT-_2"
-		(at 134.62 107.95 0)
+	(label "GND"
+		(at 133.35 107.95 0)
 		(effects
 			(font
@@
 		)
 	)
-	(label "PV+_1"
+	(label "solar_array_output_1"
 		(at 200.66 36.83 0)
 		(effects
@@
 		)
 	)
-	(label "MPPT-_2"
+	(label "GND"
 		(at 252.73 33.02 0)
 		(effects
@@
 		)
 	)
-	(label "PV-_1"
+	(label "GND"
 		(at 200.66 39.37 0)
 		(effects
@@
 	(symbol
 		(lib_id "Device:Fuse")
-		(at 133.35 119.38 180)
+		(at 132.08 119.38 180)
 		(unit 1)
 		(exclude_from_sim no)
@@
 		(dnp no)
 		(property "Reference" "Fuse_3"
-			(at 138.43 118.364 0)
+			(at 137.16 118.364 0)
 			(effects
 				(font
@@
 		)
 		(property "Value" "60A"
-			(at 138.43 120.142 0)
+			(at 137.16 120.142 0)
 			(effects
 				(font
@@
 		)
 		(property "Footprint" ""
-			(at 135.128 119.38 90)
+			(at 133.858 119.38 90)
 			(effects
 				(font
@@
 		)
 		(property "Datasheet" "~"
-			(at 133.35 119.38 0)
+			(at 132.08 119.38 0)
 			(effects
 				(font
@@
 		)
 		(property "Description" "Fuse"
-			(at 133.35 119.38 0)
-			(effects
-				(font
+			(at 132.08 119.38 0)
+			(effects
+				(font
