File: KiCad/Sensor Reader V4_JLC/Sensor Reader V4_JLC.kicad_sch (KiCad schematic)
At the start: 33 parts, among them J1 ADS1115_HE_Reader, J10 Conn_01x02_Socket, J11 Conn_01x02_Socket, J12 Conn_01x02_Socket, J13 Conn_01x02_Socket, J14 Conn_01x02_Socket, J15 5V_Input, J16 3.3V_Output, J17 Connector, USB-TYPE-C-16P, J2 ADS1115_Battery_Voltage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

Commit message: custom perf hole footprint
Parts:
- J3: footprint (none) -> Connector_Wire:SolderWire-0.5sqmm_1x06_P4.8mm_D0.9mm_OD2.3mm
- J4: footprint (none) -> Connector_Wire:SolderWire-0.1sqmm_1x06_P3.6mm_D0.4mm_OD1mm
- J6: footprint (none) -> Connector_PinHeader_1.00mm:PinHeader_1x06_P1.00mm_Vertical
Changed lines of the file:
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@@
 			)
 		)
-		(property "Footprint" ""
+		(property "Footprint" "Connector_Wire:SolderWire-0.5sqmm_1x06_P4.8mm_D0.9mm_OD2.3mm"
 			(at 236.22 81.28 0)
 			(effects
@@
 			)
 		)
-		(property "Footprint" ""
+		(property "Footprint" "Connector_Wire:SolderWire-0.1sqmm_1x06_P3.6mm_D0.4mm_OD1mm"
 			(at 259.08 81.28 0)
 			(effects
@@
 			)
 		)
-		(property "Footprint" ""
+		(property "Footprint" "Connector_PinHeader_1.00mm:PinHeader_1x06_P1.00mm_Vertical"
 			(at 158.75 181.61 0)
 			(effects
