File: KiCad/Sensor Reader V4/Sensor Reader V4.kicad_sch (KiCad schematic)
At the start: 21 parts, among them J1 ADS1115_2, J2 ADS1115_1, J3 I2C Shifter High, J4 I2C Shifter Low, J5 USB_C_Receptacle_USB2.0_16P, J6 Exposed_UART, SW1 SW_MEC_5E, SW2 SW_MEC_5E, U1 AMS1117-3.3, U2 USBLC6-2P6, U3 ESP32-S3-WROOM-1, Y1 TXC-7C

Commit message: v4_jlc test edition
Parts:
- removed U3: ESP32-S3-WROOM-1, RF_Module:ESP32-S3-WROOM-1, symbol RF_Module:ESP32-S3-WROOM-1
- removed Y1: TXC-7C, Oscillator:Oscillator_SMD_TXC_7C-4Pin_5.0x3.2mm, symbol Oscillator:TXC-7C
- added C6: 0.1uF, symbol Device:C
- added J10, J11, J12, J13, J14, J7, J8, J9: Conn_01x02_Socket, symbol Connector:Conn_01x02_Socket
- added J15: 5V_Input, symbol Connector:Conn_01x02_Socket
- added J16: 3.3V_Output, symbol Connector:Conn_01x02_Socket
- added R5, R6: 10K, symbol Device:R
- added U4: ESP32-C3-WROOM-02, RF_Module:ESP32-C3-WROOM-02, symbol RF_Module:ESP32-C3-WROOM-02
- J1: value ADS1115_2 -> ADS1115_HE_Reader
- J2: value ADS1115_1 -> ADS1115_Battery_Voltage
Connections:
- net +3.3V: now also C6.1, J16.1 (Pin_1), R5.1, R6.1, U4.1 (3V3)
- net +5V: now also J6.4 (Pin_4), J15.1 (Pin_1); no longer J6.1 (Pin_1)
- net A2_1: now also J13.1 (Pin_1)
- net A3_1: now also J14.1 (Pin_1)
- net BOOT: now also U4.8 (IO9)
- net EN: now also U4.2 (EN)
- net GND: now also J6.1 (Pin_1), C6.2, J10.2 (Pin_2), J11.2 (Pin_2), J12.2 (Pin_2), J13.2 (Pin_2), J14.2 (Pin_2), J15.2 (Pin_2), J16.2 (Pin_2), J7.2 (Pin_2), J8.2 (Pin_2), J9.2 (Pin_2), U4.19 (GND), U4.9 (GND); no longer J6.2 (Pin_2)
- net RX: now also J6.2 (Pin_2), U4.11 (IO20/RXD); no longer J6.3 (Pin_3)
- net SCL: now also U4.4 (IO5)
- net SDA: now also U4.3 (IO4)
- net TX: now also J6.3 (Pin_3), U4.12 (IO21/TXD); no longer J6.4 (Pin_4)
- net USB_D+: now also U4.14 (IO19)
- net USB_D-: now also U4.13 (IO18)
- net A0_0 renamed MPPT_Out/Batt1_In
- net MPPT_Out/Batt1_In: now also J9.1 (Pin_1)
- net A0_1 renamed Batt1_V
- net Batt1_V: now also J7.1 (Pin_1)
- net A1_0 renamed Load_In/Batt1_Out
- net Load_In/Batt1_Out: now also J10.1 (Pin_1)
- net A1_1 renamed Batt2_V
- net Batt2_V: now also J8.1 (Pin_1)
- net A2_0 renamed Batt1_Net/Batt2_In
- net Batt1_Net/Batt2_In: now also J11.1 (Pin_1)
- net A3_0 renamed Batt2_Net/Batt2_Out
- net Batt2_Net/Batt2_Out: now also J12.1 (Pin_1)
- net ALRT_0: no longer names the net of J1.6 (Pin_6)
- net ALRT_1: no longer names the net of J2.6 (Pin_6)
- new net: R6.2, U4.7 (IO8)
- new net: R5.2, U4.16 (IO2)
- no-connect marks 35 -> 14
Other:
- note added: "ADDR_0"
- note added: "ADDR_1"
- note added: "ADS1115_0_HE_Sensor_Socket"
- note added: "ADS1115_1_Battery_Voltage_Socket"
- note added: "ADS1115_1_Extra_ADC_Socket"
- note added: "Power_Connector"
- moved on the sheet: J1, J2, J6

Commit message: i
Parts:
- removed J1: ADS1115_HE_Reader, symbol Connector:Conn_01x10_Socket
- removed J2: ADS1115_Battery_Voltage, symbol Connector:Conn_01x10_Socket
- added C10, C11, C9: 10nF, symbol Device:C_Small_US
- added C5: 10uF, symbol Device:C_Small_US
- added C7, C8: 1uF, symbol Device:C_Small_US
- added R7: 10K, symbol Device:R
- added U3: ADS8688, Package_SO:TSSOP-38_4.4x9.7mm_P0.5mm, symbol Analog_ADC:ADS8688
Connections:
- net +3.3V: now also C9.2, R7.1, U3.34 (DVDD)
- net +5V: now also C10.1, C11.1, U3.30 (AVDD), U3.9 (AVDD)
- net Batt1_Net/Batt2_In: now also U3.21 (AIN_2P)
- net Batt1_V: now also U3.25 (AIN_4P)
- net Batt2_Net/Batt2_Out: now also U3.23 (AIN_3P)
- net Batt2_V: now also U3.27 (AIN_5P)
- net GND: now also C10.2, C11.2, C5.2, C7.2, C8.2, C9.1, U3.10 (AUX_IN), U3.11 (AUX_GND), U3.12 (AIN_6P), U3.13 (AIN_6GND), U3.14 (AIN_7P), U3.15 (AIN_7GND), U3.17 (AIN_0GND), U3.19 (AIN_1GND), U3.20 (AIN_2GND), U3.22 (AIN_3GND), U3.24 (AIN_4GND), U3.26 (AIN_5GND), U3.28 (AGND), U3.29 (AGND), U3.3 (DAISY), U3.31 (AGND), U3.32 (AGND), U3.33 (DGND), U3.4 (~{REFSEL}), U3.6 (REFGND), U3.8 (AGND)
- net Load_In/Batt1_Out: now also U3.18 (AIN_1P)
- net MPPT_Out/Batt1_In: now also U3.16 (AIN_0P)
- net SCL: no longer U4.4 (IO5)
- net SDA: no longer U4.3 (IO4)
- net GPIO3: now reaches U4.15 (IO3)
- net GPIO3: now also R7.2, U3.2 (~{RST/PD})
- new net: C5.1, U3.5 (REFIO)
- new net: C7.1, C8.1, U3.7 (REFCAP)
- new net CS: U3.38 (~{CS})
- new net SCLK: U3.37 (SCLK)
- new net SDI: U3.1 (SDI)
- new net SDO: U3.36 (SDO)
- no-connect marks 14 -> 13
Other:
- note removed: "ADDR_0"
- note removed: "ADDR_1"
- note removed: "ADS1115 External Module"
- moved on the sheet: C6, J10, J11, J12, J13, J14, J7, J8, J9, R5, R6, U4

Commit message: finish populating components
Parts:
- removed C1: 47uF, symbol Device:C_Polarized
- removed C10, C11, C9: 10nF, symbol Device:C_Small_US
- removed C2: 100uF, symbol Device:C_Polarized
- removed C3: 4.7uF, symbol Device:C_Polarized
- removed C4: 100nF, symbol Device:C
- removed C5: 10uF, symbol Device:C_Small_US
- removed C6: 0.1uF, symbol Device:C
- removed C7, C8: 1uF, symbol Device:C_Small_US
- removed J3: I2C Shifter High, symbol Connector:Conn_01x06_Socket
- removed J4: I2C Shifter Low, symbol Connector:Conn_01x06_Socket
- removed J5: USB_C_Receptacle_USB2.0_16P, symbol Connector:USB_C_Receptacle_USB2.0_16P
- removed R1, R2: 5.1K, symbol Device:R
- removed R3, R4, R5, R6, R7: 10K, symbol Device:R
- added C1: 47uF, PCM_JLCPCB:C_0805, symbol PCM_JLCPCB-Capacitors:0805,47uF
- added C10, C11, C5, C9: 10nF, PCM_JLCPCB:C_0603, symbol PCM_JLCPCB-Capacitors:0603,10nF
- added C12, C4, C6: 100nF, PCM_JLCPCB:C_0603, symbol PCM_JLCPCB-Capacitors:0603,100nF
- added C3: 4.7uF, PCM_JLCPCB:C_0603, symbol PCM_JLCPCB-Capacitors:0603,4.7uF
- added C7, C8: 1uF, PCM_JLCPCB:C_0603, symbol PCM_JLCPCB-Capacitors:0603,1uF
- added J1: USB_C_Receptacle_USB2.0_16P, Connector_USB:USB_C_Receptacle_Palconn_UTC16-G, symbol Connector:USB_C_Receptacle_USB2.0_16P
- added R1, R2: 5.1Ω, PCM_JLCPCB:R_0603, symbol PCM_JLCPCB-Resistors:0603,5.1Ω
- added R10, R11, R12, R13, R8, R9: 1kΩ, PCM_JLCPCB:R_0603, symbol PCM_JLCPCB-Resistors:0603,1kΩ
- added R16, R18: 100kΩ, PCM_JLCPCB:R_0603, symbol PCM_JLCPCB-Resistors:0603,100kΩ
- added R17, R19: 20kΩ, PCM_JLCPCB:R_0603, symbol PCM_JLCPCB-Resistors:0603,20kΩ
- added R3, R4, R5, R6, R7: 10kΩ, PCM_JLCPCB:R_0603, symbol PCM_JLCPCB-Resistors:0603,10kΩ
- J10: value Conn_01x02_Socket -> L_I/B1_Out; footprint (none) -> Connector_JST:JST_XH_B2B-XH-A_1x02_P2.50mm_Vertical
- J11: value Conn_01x02_Socket -> B1_Net/B2_In; footprint (none) -> Connector_JST:JST_XH_B2B-XH-A_1x02_P2.50mm_Vertical
- J12: value Conn_01x02_Socket -> B2_Net/B2_Out; footprint (none) -> Connector_JST:JST_XH_B2B-XH-A_1x02_P2.50mm_Vertical
- J13: value Conn_01x02_Socket -> AIN_4; footprint (none) -> Connector_JST:JST_XH_B2B-XH-A_1x02_P2.50mm_Vertical
- J14: value Conn_01x02_Socket -> AIN_5; footprint (none) -> Connector_JST:JST_XH_B2B-XH-A_1x02_P2.50mm_Vertical
- J15: footprint (none) -> Connector_JST:JST_XH_B2B-XH-A_1x02_P2.50mm_Vertical
- J16: footprint (none) -> Connector_PinHeader_2.54mm:PinHeader_1x02_P2.54mm_Vertical
- J6: footprint (none) -> Connector_PinHeader_2.54mm:PinHeader_1x06_P2.54mm_Vertical
- J7: value Conn_01x02_Socket -> Batt1_V; footprint (none) -> Connector_JST:JST_XH_B2B-XH-A_1x02_P2.50mm_Vertical
- J8: value Conn_01x02_Socket -> Batt2_V; footprint (none) -> Connector_JST:JST_XH_B2B-XH-A_1x02_P2.50mm_Vertical
- J9: value Conn_01x02_Socket -> M_OUT/B1_In; footprint (none) -> Connector_JST:JST_XH_B2B-XH-A_1x02_P2.50mm_Vertical
- SW1: value SW_MEC_5E -> BOOT_Btn; footprint Button_Switch_SMD:SW_MEC_5GSH9 -> PCM_JLCPCB:SW-SMD_4P-L5.1-W5.1-P3.70-LS6.5-TL-2
- SW2: value SW_MEC_5E -> EN_Btn; footprint Button_Switch_SMD:SW_MEC_5GSH9 -> PCM_JLCPCB:SW-SMD_4P-L5.1-W5.1-P3.70-LS6.5-TL-2
Connections:
- net A2_1 is gone; now on net GND: J13.1 (Pin_1)
- net A3_1 is gone; now on net GND: J14.1 (Pin_1)
- net +3.3V: now also J16.2 (Pin_2), C11.1, C12.2, C3.1, C6.1, R3.1, R4.1, R5.1, R6.1, R7.2; no longer J16.1 (Pin_1)
- net +5V: now also J15.2 (Pin_2), C1.1, C10.1, C9.1; no longer J15.1 (Pin_1)
- net BOOT: now also SW1.1, SW1.2, R4.2; no longer SW2.1, SW2.2
- net Batt1_Net/Batt2_In: now also J11.2 (Pin_2), R10.1; no longer J11.1 (Pin_1), U3.21 (AIN_2P)
- net Batt1_V: now also J7.2 (Pin_2), R16.1; no longer J7.1 (Pin_1), U3.25 (AIN_4P)
- net Batt2_Net/Batt2_Out: now also J12.2 (Pin_2), R11.1; no longer J12.1 (Pin_1), U3.23 (AIN_3P)
- net Batt2_V: now also J8.2 (Pin_2), R18.1; no longer J8.1 (Pin_1), U3.27 (AIN_5P)
- net CS: now also U4.6 (IO7)
- net EN: now also SW2.1, SW2.2, C4.1, R3.2; no longer SW1.1, SW1.2
- net GND: now also J10.1 (Pin_1), J11.1 (Pin_1), J12.1 (Pin_1), J15.1 (Pin_1), J16.1 (Pin_1), J7.1 (Pin_1), J8.1 (Pin_1), J9.1 (Pin_1), C1.2, C10.2, C11.2, C12.1, C3.2, C4.2, C5.2, C6.2, C7.2, C8.2, C9.2, J1.A1 (GND), J1.A12 (GND), J1.B1 (GND), J1.B12 (GND), J1.S1 (SHIELD), R1.2, R17.2, R19.2, R2.2; no longer J10.2 (Pin_2), J11.2 (Pin_2), J12.2 (Pin_2), J13.2 (Pin_2), J14.2 (Pin_2), J15.2 (Pin_2), J16.2 (Pin_2), J7.2 (Pin_2), J8.2 (Pin_2), J9.2 (Pin_2), U3.12 (AIN_6P), U3.14 (AIN_7P)
- net Load_In/Batt1_Out: now also J10.2 (Pin_2), R9.1; no longer J10.1 (Pin_1), U3.18 (AIN_1P)
- net MPPT_Out/Batt1_In: now also J9.2 (Pin_2), R8.1; no longer J9.1 (Pin_1), U3.16 (AIN_0P)
- net SCLK: now also U4.5 (IO6)
- net SDI: now also U4.4 (IO5)
- net SDO: now also U4.3 (IO4)
- net USB_D+: now also J1.A6 (D+), J1.B6 (D+)
- net USB_D-: now also J1.A7 (D-), J1.B7 (D-)
- net at U3.5 (REFIO): now also C5.1
- net at U3.7 (REFCAP): now also C7.1, C8.1
- net at D1.2 (A): now also J1.A4 (VBUS), J1.A9 (VBUS), J1.B4 (VBUS), J1.B9 (VBUS)
- net at U4.7 (IO8): now also R6.2
- net at U4.16 (IO2): now also R5.2
- net GPIO3 renamed RST
- net RST: now also R7.1
- new net: R11.2, U3.23 (AIN_3P)
- new net: R18.2, R19.1, U3.14 (AIN_7P)
- new net: R10.2, U3.21 (AIN_2P)
- new net: R16.2, R17.1, U3.12 (AIN_6P)
- new net: R8.2, U3.16 (AIN_0P)
- new net: R9.2, U3.18 (AIN_1P)
- new net: R12.2, U3.25 (AIN_4P)
- new net: R13.2, U3.27 (AIN_5P)
- new net: J1.A5 (CC1), R1.1
- new net: J1.B5 (CC2), R2.1
- new net AIN_4: J13.2 (Pin_2), R12.1
- new net AIN_5: J14.2 (Pin_2), R13.1
- no-connect marks 13 -> 5
Other:
- note added: "ADS8688"
- note added: "Battery_Voltage_Socket"
- note added: "ESP32_C3_WROOM (With Antenna)"
- note added: "Extra_ADC_Socket"
- note added: "HE_Sensor_Socket"
- note removed: "ADS1115_0_HE_Sensor_Socket"
- note removed: "ADS1115_1_Battery_Voltage_Socket"
- note removed: "ADS1115_1_Extra_ADC_Socket"
- note removed: "I2C Level Shifter (5 hole length, 2.54mm * 3 gap)"
- moved on the sheet: J10, J11, J12, J13, J14, J15, J16, J6, J7, J8, J9, U2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

Commit message: data coll
Parts:
- removed U2: USBLC6-2P6, Package_TO_SOT_SMD:SOT-666, symbol Power_Protection:USBLC6-2P6
- J1: footprint Connector_USB:USB_C_Receptacle_Palconn_UTC16-G -> (none)
Connections:
- net GND: now also J1.SH (SHIELD); no longer J1.S1 (SHIELD)

Commit message: pdb
Parts:
- removed C1: 47uF, PCM_JLCPCB:C_0805, symbol PCM_JLCPCB-Capacitors:0805,47uF
- removed C12: 100nF, PCM_JLCPCB:C_0603, symbol PCM_JLCPCB-Capacitors:0603,100nF
- removed D1: 1N5819WS, Diode_SMD:D_SOD-323, symbol Diode:1N5819WS
- removed J1: USB_C_Receptacle_USB2.0_16P, symbol Connector:USB_C_Receptacle_USB2.0_16P
- removed U1: AMS1117-3.3, Package_TO_SOT_SMD:SOT-223-3_TabPin2, symbol Regulator_Linear:AMS1117-3.3
- removed U4: ESP32-C3-WROOM-02, RF_Module:ESP32-C3-WROOM-02, symbol RF_Module:ESP32-C3-WROOM-02
- added C12, C20: 10uF, Capacitor_SMD:C_0603_1608Metric_Pad1.08x0.95mm_HandSolder, symbol PCM_JLCPCB-Capacitors:0603,10nF
- added C13, C2: 1uF, Capacitor_SMD:C_0603_1608Metric_Pad1.08x0.95mm_HandSolder, symbol PCM_JLCPCB-Capacitors:0805,47uF
- added C14, C15, C16, C17, C18, C19, C21, C22: 4.7nF, Capacitor_SMD:C_0603_1608Metric_Pad1.08x0.95mm_HandSolder, symbol SamacSys_Parts:C_45deg
- added C23: 10uF, Capacitor_SMD:C_0603_1608Metric_Pad1.08x0.95mm_HandSolder, symbol PCM_JLCPCB-Capacitors:0603,100nF
- added IC1: TLV76733DGNR, SamacSys_Parts:SOP65P490X110-9N, symbol SamacSys_Parts:TLV76733DGNR
- added IC2: ESP32-C3-WROOM-02-H4, SamacSys_Parts:ESP32C3WROOM02H4, symbol SamacSys_Parts:ESP32-C3-WROOM-02-H4
- added J2: UJ20-C-H-G-MSMT-2B-P16-TR, SamacSys_Parts:UJ20CHGMSMT2BP16TR, symbol SamacSys_Parts:UJ20-C-H-G-MSMT-2B-P16-TR
- added R14, R15: 1kΩ, Resistor_SMD:R_0603_1608Metric_Pad0.98x0.95mm_HandSolder, symbol PCM_JLCPCB-Resistors:0603,1kΩ
- added TP1, TP2, TP3, TP4, TP5, TP6, TP7, TP8: TestPoint, TestPoint:TestPoint_Pad_D1.0mm, symbol Connector:TestPoint
- C10, C9: value 10nF -> 1uF; footprint PCM_JLCPCB:C_0603 -> Capacitor_SMD:C_0603_1608Metric_Pad1.08x0.95mm_HandSolder
- C11: value 10nF -> 10uF; footprint PCM_JLCPCB:C_0603 -> Capacitor_SMD:C_0805_2012Metric_Pad1.18x1.45mm_HandSolder
- C3, C6, C7: footprint PCM_JLCPCB:C_0603 -> Capacitor_SMD:C_0603_1608Metric_Pad1.08x0.95mm_HandSolder
- C4: value 100nF -> 1uF; footprint PCM_JLCPCB:C_0603 -> Capacitor_SMD:C_0603_1608Metric_Pad1.08x0.95mm_HandSolder
- C5: value 10nF -> 10uF; footprint PCM_JLCPCB:C_0603 -> Capacitor_SMD:C_0603_1608Metric_Pad1.08x0.95mm_HandSolder
- C8: value 1uF -> 10uF; footprint PCM_JLCPCB:C_0603 -> Capacitor_SMD:C_0603_1608Metric_Pad1.08x0.95mm_HandSolder
- R1, R10, R11, R12, R13, R16, R17, R18, R19, R2, R3, R4, R5, R6, R7, R8, R9: footprint PCM_JLCPCB:R_0603 -> Resistor_SMD:R_0603_1608Metric_Pad0.98x0.95mm_HandSolder
- SW1, SW2: footprint PCM_JLCPCB:SW-SMD_4P-L5.1-W5.1-P3.70-LS6.5-TL-2 -> SamacSys_Parts:TS0266100BK100LCRD
- U3: footprint Package_SO:TSSOP-38_4.4x9.7mm_P0.5mm -> SamacSys_Parts:SOP50P640X120-38N
Connections:
- net +3.3V: now also C13.1, C23.1, IC1.1 (OUT), IC1.2 (SNS), IC2.1 (3V3), TP1.1
- net +5V: now also C12.1, C2.1, C20.1, IC1.5 (EN), IC1.8 (IN), J2.A4 (VBUS_1), J2.B4 (VBUS_2), TP3.1
- net BOOT: now also IC2.8 (IO9)
- net CS: now also IC2.6 (IO7), TP4.1
- net EN: now also IC2.2 (EN)
- net GND: now also C12.2, C13.2, C14.1, C15.1, C16.1, C17.1, C18.1, C19.1, C2.2, C20.2, C21.1, C22.1, C23.2, IC1.4 (GND_1), IC1.6 (GND_2), IC1.9 (EP), IC2.19 (GND_2), IC2.20 (GND_3), IC2.21 (GND_4), IC2.22 (GND_5), IC2.23 (GND_6), IC2.24 (GND_7), IC2.25 (GND_8), IC2.26 (GND_9), IC2.27 (GND_10), IC2.9 (GND_1), J2.A1 (GND_1), J2.B1 (GND_2), J2.MH1, J2.MH2, J2.MH3, J2.MH4, TP2.1, TP8.1
- net RST: now also IC2.15 (IO3)
- net RX: now also IC2.11 (RXD)
- net SCLK: now also IC2.5 (IO6), TP5.1
- net SDI: now also IC2.4 (IO5), TP6.1
- net SDO: now also IC2.3 (IO4), TP7.1
- net TX: now also IC2.12 (TXD)
- net USB_D+: now also IC2.14 (IO19), J2.A6 (DP1), J2.B6 (DP2)
- net USB_D-: now also IC2.13 (IO18), J2.A7 (DN1), J2.B7 (DN2)
- net at R11.2, U3.23 (AIN_3P): now also C18.2
- net at R18.2, R19.1: now also R15.1; no longer U3.14 (AIN_7P)
- net at R10.2, U3.21 (AIN_2P): now also C17.2
- net at R16.2, R17.1: now also R14.1; no longer U3.12 (AIN_6P)
- net at R8.2, U3.16 (AIN_0P): now also C21.2
- net at R9.2, U3.18 (AIN_1P): now also C22.2
- net at R12.2, U3.25 (AIN_4P): now also C19.2
- net at R13.2, U3.27 (AIN_5P): now also C14.2
- net at R5.2: now also IC2.16 (IO2)
- net at R1.1: now also J2.B5 (CC2)
- net at R2.1: now also J2.A5 (CC1)
- net at R6.2: now also IC2.7 (IO8)
- new net: C15.2, R14.2, U3.12 (AIN_6P)
- new net: C16.2, R15.2, U3.14 (AIN_7P)
- no-connect marks 5 -> 7
Other:
- note added: "TLV767-Fixed 3.3 Voltage Regulator"
- note removed: "AMS1117-3.3 Voltage Regulator"
- moved on the sheet: C10, C11, C9, R1, R10, R11, R12, R13, R16, R17, R18, R19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

Commit message: KICAD pcb
Parts:
- removed J2: UJ20-C-H-G-MSMT-2B-P16-TR, SamacSys_Parts:UJ20CHGMSMT2BP16TR, symbol SamacSys_Parts:UJ20-C-H-G-MSMT-2B-P16-TR
- removed R1: 5.1Ω, Resistor_SMD:R_0603_1608Metric_Pad0.98x0.95mm_HandSolder, symbol PCM_JLCPCB-Resistors:0603,5.1Ω
- removed TP8: TestPoint, TestPoint:TestPoint_Pad_D1.0mm, symbol Connector:TestPoint
- added J1: 10172013-00011LF, 1017201300011LF, symbol SamacSys_Parts:10172013-00011LF
- added R20: 5.1Ω, Resistor_SMD:R_0603_1608Metric_Pad0.98x0.95mm_HandSolder, symbol PCM_JLCPCB-Resistors:0603,5.1Ω
Connections:
- net +5V: now also J1.A4 (VBUS_1), J1.A9 (VBUS_2)
- net GND: now also J1.1 (MH1), J1.2 (MH2), J1.3 (MH3), J1.4 (MH4), J1.A1 (GND_1), J1.A12 (GND_2), R20.2
- net USB_D+: now also J1.A6 (DP1), J1.B6 (DP2)
- net USB_D-: now also J1.A7 (DN1), J1.B7 (DN2)
- net at R2.1: now also J1.A5 (CC1)
- new net: J1.B5 (CC2), R20.1

Commit message: final pcb design
Parts:
- removed J1: 10172013-00011LF, 1017201300011LF, symbol SamacSys_Parts:10172013-00011LF
- added J1: USB_C_Receptacle_USB2.0_16P, Connector_USB:USB_C_Receptacle_XKB_U262-16XN-4BVC11, symbol Connector:USB_C_Receptacle_USB2.0_16P
- added J2: GPIO, Connector_PinHeader_2.54mm:PinHeader_1x03_P2.54mm_Vertical, symbol Connector:Conn_01x03_Socket
- R2, R20: value 5.1Ω -> 5.1KΩ
Connections:
- net +5V: now also J1.A4 (VBUS), J1.A9 (VBUS), J1.B4 (VBUS), J1.B9 (VBUS)
- net GND: now also R2.1, J1.A1 (GND), J1.A12 (GND), J1.B1 (GND), J1.B12 (GND), J1.SH (SHIELD); no longer R2.2
- net USB_D+: now also J1.A6 (D+), J1.B6 (D+)
- net USB_D-: now also J1.A7 (D-), J1.B7 (D-)
- net at R20.1: now also J1.B5 (CC2)
- net GPIO10: now reaches IC2.10 (IO10)
- net GPIO10: now also J2.3 (Pin_3)
- net GPIO1: now reaches IC2.17 (IO1)
- net GPIO1: now also J2.2 (Pin_2)
- net GPIO0: now reaches IC2.18 (IO0)
- net GPIO0: now also J2.1 (Pin_1)
- new net: J1.A5 (CC1), R2.2
- no-connect marks 7 -> 4
Other:
- note added: "Extra"
